File: GemToasterAmp.kicad_sch (KiCad schematic)
At the start: 12 parts

Commit message: 57rty
Parts:
- added C? (x2): 100n, Capacitor_SMD:C_0805_2012Metric_Pad1.18x1.45mm_HandSolder, symbol 000_Capacitor_Film_Immo:cap_film_0805
- added C?: 470n, Capacitor_SMD:C_0805_2012Metric_Pad1.18x1.45mm_HandSolder, symbol 000_Capacitor_Film_Immo:cap_film_0805
- added C?: 100p, Capacitor_SMD:C_0805_2012Metric_Pad1.18x1.45mm_HandSolder, symbol 000_Capacitor_Film_Immo:cap_film_0805
- added C? (x2): 15n, Capacitor_SMD:C_0805_2012Metric_Pad1.18x1.45mm_HandSolder, symbol 000_Capacitor_Film_Immo:cap_film_0805
- added EC? (x2): 10u, Capacitor_SMD:CP_Elec_6.3x5.9, symbol 000_Capacitor_Electrolytic_Immo:10u
- added EC? (x2): 220u, Capacitor_SMD:CP_Elec_10x10, symbol 000_Capacitor_Electrolytic_Immo:220u
- added PT?: B250k, Potentiometer_THT:Potentiometer_Alpha_RD901F-40-00D_Single_Vertical_CircularHoles, symbol 000_Resistors_Immo:Potentiometer
- added PT?: B10k, Potentiometer_THT:Potentiometer_Alpha_RD901F-40-00D_Single_Vertical_CircularHoles, symbol 000_Resistors_Immo:Potentiometer
- added PT?: B100k, Potentiometer_THT:Potentiometer_Alpha_RD901F-40-00D_Single_Vertical_CircularHoles, symbol 000_Resistors_Immo:Potentiometer
- added PT?: B5k, Potentiometer_THT:Potentiometer_Alpha_RD901F-40-00D_Single_Vertical_CircularHoles, symbol 000_Resistors_Immo:Potentiometer
- added Q? (x2): 2N5457/J201, Package_TO_SOT_SMD:SOT-23, symbol Transistor_FET:MMBFJ112
- added R? (x2): 3k9, Resistor_SMD:R_0805_2012Metric_Pad1.20x1.40mm_HandSolder, symbol 000_Resistors_Immo:Resistor_0805
- added R? (x2): 2M2, Resistor_SMD:R_0805_2012Metric_Pad1.20x1.40mm_HandSolder, symbol 000_Resistors_Immo:Resistor_0805
- added R?: 24k, Resistor_SMD:R_0805_2012Metric_Pad1.20x1.40mm_HandSolder, symbol 000_Resistors_Immo:Resistor_0805
- added R?: 12k, Resistor_SMD:R_0805_2012Metric_Pad1.20x1.40mm_HandSolder, symbol 000_Resistors_Immo:Resistor_0805
- added R?: 4k7, Resistor_SMD:R_0805_2012Metric_Pad1.20x1.40mm_HandSolder, symbol 000_Resistors_Immo:Resistor_0805
- added R?: 470k, Resistor_SMD:R_0805_2012Metric_Pad1.20x1.40mm_HandSolder, symbol 000_Resistors_Immo:Resistor_0805
Connections:
- net GND: now also U?.3 (+), U?.4 (GND), C?.1, C?.2, C?.2, EC?.2, PT?.1, PT?.1, R?.2, R?.2, R?.2, R?.2, R?.2, R?.2
- net VCC: now also U?.6 (V+), C?.1, EC?.1, Q?.1 (D), R?.1
- net at U?.1 (GAIN): now also PT?.1
- net at U?.2 (-): now also PT?.2
- net at U?.5: now also EC?.1
- net at U?.7 (BYPASS): now also C?.2
- net at U?.8 (GAIN): now also PT?.2, PT?.3
- net at C?.2: now also C?.2, R?.1
- new net: C?.1, Q?.1 (D), R?.2
- new net: EC?.1, Q?.2 (S), R?.1 (x2)
- new net: C?.2, Q?.3 (G), R?.1
- new net: C?.1, PT?.1, R?.2
- new net: C?.1, PT?.2
- new net: C?.1, PT?.3, R?.1
- new net: EC?.2, PT?.3
- new net: PT?.2, Q?.3 (G), R?.1
- new net: C?.2, PT?.3
- new net: EC?.2, R?.1
- new net SPKR+: EC?.2
Other:
- note added: "Not sure about this bit, seems odd to me"
- moved on the sheet: C?, D?, EC?, Q?, R?, U?

Commit message: vjghdfjghf
Parts:
- removed C?: 100p, Capacitor_SMD:C_0805_2012Metric_Pad1.18x1.45mm_HandSolder, symbol 000_Capacitor_Film_Immo:cap_film_0805
- removed EC?: 220u, Capacitor_SMD:CP_Elec_10x10, symbol 000_Capacitor_Electrolytic_Immo:220u
- added C7: 100p, Capacitor_SMD:C_0805_2012Metric_Pad1.18x1.45mm_HandSolder, symbol 000_Capacitor_Film_Immo:cap_film_0805
- added EC5: 220u, Capacitor_SMD:CP_Elec_10x10, symbol 000_Capacitor_Electrolytic_Immo:220u
- added J?: Speaker(2-8 ohm), TerminalBlock:TerminalBlock_Altech_AK300-2_P5.00mm, symbol Connector:Screw_Terminal_01x02
- added J?: Speaker, Connector_Molex:Molex_KK-254_AE-6410-02A_1x02_P2.54mm_Vertical, symbol 000_Connectors_Immo:2pin_molex_2.54mm_male
- added J?: Input, TerminalBlock:TerminalBlock_Altech_AK300-2_P5.00mm, symbol Connector:Screw_Terminal_01x02
- added J?: Input, Connector_Molex:Molex_KK-254_AE-6410-02A_1x02_P2.54mm_Vertical, symbol 000_Connectors_Immo:2pin_molex_2.54mm_male
- added J?: Battery, TerminalBlock:TerminalBlock_Altech_AK300-2_P5.00mm, symbol Connector:Screw_Terminal_01x02
- added J?: Battery, Connector_Molex:Molex_KK-254_AE-6410-02A_1x02_P2.54mm_Vertical, symbol 000_Connectors_Immo:2pin_molex_2.54mm_male
- added J?: StompQC, symbol 000_Pin_Headers_Immo:StompQC
- added SW?: Power, symbol 000_Switches_Immo:SW_SPDT
- gave numbers to parts that had none: 34
Connections:
- net +BATT: now also J?.2 (Pin_2), J?.2 (Pin_2), J?.2 (Vin), SW?.2 (B); no longer D1.2 (A)
- net GND: now also C7.2, EC5.2, J?.1 (Pin_1), J?.1 (Pin_1), J?.1 (Pin_1), J?.1 (Pin_1), J?.1 (Pin_1), J?.1 (Pin_1), J?.3 (GND)
- net INPUT: now also J?.1 (In), J?.2 (Pin_2), J?.2 (Pin_2)
- net SPKR+: now also J?.2 (Pin_2), J?.2 (Pin_2), J?.4 (Out)
- net VCC: now also C7.1, EC5.1
- new net: D1.2 (A), SW?.1 (A)
- no-connect marks 0 -> 1
Other:
- note added: "Add switched jack for battery"
- note removed: "Not sure about this bit, seems odd to me"
- moved on the sheet: D1, D2, D3, R13

Commit message: dgfhfgh
Parts:
- removed J?: Battery, Connector_Molex:Molex_KK-254_AE-6410-02A_1x02_P2.54mm_Vertical, symbol 000_Connectors_Immo:2pin_molex_2.54mm_male
- added BT1: 9v Battery, Battery:BatteryHolder_Eagle_12BH611-GR, symbol Device:Battery
- added J7: AudioJack3_Switch, Connector_Audio:Jack_6.35mm_Neutrik_NMJ6HFD2_Horizontal, symbol Connector:AudioJack3_Switch
- added J?: GND, Connector_Molex:Molex_KK-254_AE-6410-02A_1x02_P2.54mm_Vertical, symbol 000_Connectors_Immo:2pin_molex_2.54mm_male
- added J?: Vcc, Connector_Molex:Molex_KK-254_AE-6410-02A_1x02_P2.54mm_Vertical, symbol 000_Connectors_Immo:2pin_molex_2.54mm_male
- added JP1: batt/DC, Jumper:SolderJumper-3_P1.3mm_Bridged12_RoundedPad1.0x1.5mm, symbol 000_Connectors_Immo:Jumper_3_Bridged12
- added JP2: Disable Batt Disconnect, Jumper:SolderJumper-2_P1.3mm_Open_RoundedPad1.0x1.5mm, symbol 000_Connectors_Immo:Jumper_2_Open
- J6: renamed from J?; value Battery -> Power
- gave numbers to parts that had none: 6
Connections:
- net +BATT: now also D1.2 (A), BT1.1 (+), JP1.3 (B); no longer J4.2 (Vin), J6.2 (Pin_2), SW1.2 (B)
- net GND: now also J7.S, J7.SN, J7.TN, J?.1 (Pin_1), J?.2 (Pin_2), JP2.1 (A)
- net INPUT: now also J7.T
- net VCC: now also SW1.1 (A), J?.1 (Pin_1), J?.2 (Pin_2); no longer D1.1 (K)
- new net -BATT: BT1.2 (-), J7.R, JP2.2 (B)
- new net Vsupp: J4.2 (Vin), J6.2 (Pin_2), JP1.2 (C)
- new net power_in: D1.1 (K), JP1.1 (A), SW1.2 (B)
- no-connect marks 1 -> 2
Other:
- note added: "Slight difference between Power & Battery Aim to avoid DC Jack putting voltage across battery."
- note added: "When Mono Plug is in, shorts: Ring to Sleeve (to GND) Disabled to always on by closing open junction"
- note removed: "Add switched jack for battery"
- moved on the sheet: J6

Commit message: layout v0.1
Parts:
- removed J4: StompQC, symbol 000_Pin_Headers_Immo:StompQC
- removed J?: GND, Connector_Molex:Molex_KK-254_AE-6410-02A_1x02_P2.54mm_Vertical, symbol 000_Connectors_Immo:2pin_molex_2.54mm_male
- removed J?: Vcc, Connector_Molex:Molex_KK-254_AE-6410-02A_1x02_P2.54mm_Vertical, symbol 000_Connectors_Immo:2pin_molex_2.54mm_male
- removed PT1: B100k, Potentiometer_THT:Potentiometer_Alpha_RD901F-40-00D_Single_Vertical_CircularHoles, symbol 000_Resistors_Immo:Potentiometer
- removed PT4: B5k, Potentiometer_THT:Potentiometer_Alpha_RD901F-40-00D_Single_Vertical_CircularHoles, symbol 000_Resistors_Immo:Potentiometer
- added J8: Vcc, Connector_PinHeader_2.54mm:PinHeader_1x02_P2.54mm_Vertical, symbol 000_Pin_Headers_Immo:Conn_01x02_Male
- added J9: GND, Connector_PinHeader_2.54mm:PinHeader_1x02_P2.54mm_Vertical, symbol 000_Pin_Headers_Immo:Conn_01x02_Male
- added JP3: SWDIR, Jumper:SolderJumper-3_P1.3mm_Bridged12_RoundedPad1.0x1.5mm, symbol 000_Connectors_Immo:Jumper_3_Bridged12
- added PT1: B100k, 000 Resistors Immo:16MM_CENTERMOUNT, symbol 000_Resistors_Immo:dual_footprint_pot
- added PT4: B5k, 000 Resistors Immo:16MM_CENTERMOUNT, symbol 000_Resistors_Immo:16mm Pot
- J1: footprint TerminalBlock:TerminalBlock_Altech_AK300-2_P5.00mm -> 000 Connectors Immo:TerminalBlock_Altech_AK300-2_P5.00mm; symbol Connector:Screw_Terminal_01x02 -> 000_Connectors_Immo:Screw_Terminal_01x02; PIN1 (none) -> GND; PIN2 (none) -> INPUT
- J2: footprint TerminalBlock:TerminalBlock_Altech_AK300-2_P5.00mm -> 000 Connectors Immo:TerminalBlock_Altech_AK300-2_P5.00mm; symbol Connector:Screw_Terminal_01x02 -> 000_Connectors_Immo:Screw_Terminal_01x02; PIN1 (none) -> GND; PIN2 (none) -> SPKR+
- J3: footprint Connector_Molex:Molex_KK-254_AE-6410-02A_1x02_P2.54mm_Vertical -> 000 Connectors Immo:Molex_KK-254_AE-6410-02A_1x02_P2.54mm_Vertical_copy; PIN1 (none) -> GND; PIN2 (none) -> Input
- J5: footprint Connector_Molex:Molex_KK-254_AE-6410-02A_1x02_P2.54mm_Vertical -> 000 Connectors Immo:Molex_KK-254_AE-6410-02A_1x02_P2.54mm_Vertical_copy; PIN1 (none) -> GND; PIN2 (none) -> SPKR+
- J6: footprint TerminalBlock:TerminalBlock_Altech_AK300-2_P5.00mm -> 000 Connectors Immo:TerminalBlock_Altech_AK300-2_P5.00mm; symbol Connector:Screw_Terminal_01x02 -> 000_Connectors_Immo:Screw_Terminal_01x02; PIN1 (none) -> GND; PIN2 (none) -> Vsupp
- PT2, PT3: footprint Potentiometer_THT:Potentiometer_Alpha_RD901F-40-00D_Single_Vertical_CircularHoles -> 000 Resistors Immo:16MM_CENTERMOUNT; symbol 000_Resistors_Immo:Potentiometer -> 000_Resistors_Immo:16mm Pot
- Q1: footprint Package_TO_SOT_SMD:SOT-23 -> 000 Transistors Immo:JFET Dual Foot; symbol Transistor_FET:MMBFJ112 -> 000_Transistors_FET_Immo:2N5457/J201
- Q2: renamed from Q3; footprint Package_TO_SOT_SMD:SOT-23 -> 000 Transistors Immo:JFET Dual Foot; symbol Transistor_FET:MMBFJ112 -> 000_Transistors_FET_Immo:2N5457/J201
- Q3: renamed from Q2; footprint Package_TO_SOT_SMD:SOT-23 -> 000 Transistors Immo:JFET Dual Foot; symbol Transistor_FET:MMBFJ112 -> 000_Transistors_FET_Immo:2N5457/J201
- SW1: value Power -> On/Off; footprint (none) -> 000 Switches Immo:SPDT_M9040P_TH; NAME (none) -> Power
- U1: footprint (none) -> 000 IC Immo:DIL8
Connections:
- net GND: now also J9.1 (Pin_1), J9.2 (Pin_2), PT1.1
- net VCC: now also J8.1 (Pin_1), J8.2 (Pin_2), JP3.2 (C); no longer SW1.1 (A)
- net at U1.1 (GAIN): now also PT4.1
- net at U1.8 (GAIN): now also PT4.2, PT4.3
- net at Q3.3 (G), R4.1: now also PT1.2
- net at C3.2: now also PT1.3
- net at SW1.3 (C): now also JP3.3 (B)
- new net: JP3.1 (A), SW1.1 (A)
- no-connect marks 2 -> 1
Other:
- moved on the sheet: BT1, C7, D1, D2, D3, EC5, J1, J2, J3, R13, SW1
