File: GemToasterAmp.kicad_pcb (KiCad board)
At the start: 2 copper layers, 105.4 x 50.8 mm, 49 parts, among them J1 Input, J2 Speaker(2-8 ohm), J3 Input, J5 Speaker, J6 Power, J7 AudioJack3_Switch, J8 Vcc, J9 GND, Q1 2N5457/J201, Q2 2N5457/J201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

Commit message: erfdrgd
Parts:
- PT1, PT2, PT3, PT4: footprint 000 Resistors Immo:16MM_CENTERMOUNT -> 000 Resistors Immo:16MM_AngleMount
- moved R3 19.1 mm to (145.1, 49.5), turned to 180 degrees
- moved PT4 12.1 mm to (209.6, 42.5), turned to 0 degrees
- moved PT3 12.1 mm to (190.5, 42.5), turned to 0 degrees
- moved PT1 12.1 mm to (171.4, 42.5), turned to 0 degrees
- moved PT2 12.1 mm to (152.4, 42.5), turned to 0 degrees
Other:
- board size 105.4 x 50.8 mm -> 105.4 x 48.9 mm

Commit message: dfgdfgg
Parts:
- added REF**: MountingHole_3.2mm_M3_Pad_Via, MountingHole:MountingHole_3.2mm_M3_Pad_Via, F.Cu at (116.8, 87.0)
- added REF**: MountingHole_3.2mm_M3_Pad_Via, MountingHole:MountingHole_3.2mm_M3_Pad_Via, F.Cu at (158.1, 54.0)
- added REF**: MountingHole_3.2mm_M3_Pad_Via, MountingHole:MountingHole_3.2mm_M3_Pad_Via, F.Cu at (214.6, 87.0)
- BT1, EC1, EC2, EC3, EC4, EC5, J1, J2, J3, J5, J6, PT1, PT2, PT3, PT4: moved to B.Cu
- D2: footprint LED_THT:LED_D5.0mm -> 000 Diodes Immo:LED_D5.0mm_Flat; moved to B.Cu
- SW1: footprint 000 Switches Immo:SPDT_M9040P_TH -> 000 Switches Immo:SPDT-100SP4T1-Right-Angle
- moved BT1 86.5 mm to (176.5, 72.4), turned to 180 degrees
- moved J2 63.6 mm to (147.9, 80.6), turned to 180 degrees
- moved J5 49.8 mm to (242.6, 107.9), turned to 0 degrees
- moved EC4 46.3 mm to (168.5, 121.3), turned to 0 degrees
- moved EC5 46.0 mm to (199.8, 116.2)
- moved R10 44.8 mm to (162.2, 112.5)
- moved R2 44.8 mm to (173.0, 112.5)
- moved R4 44.8 mm to (179.1, 112.5)
- moved C3 44.8 mm to (173.0, 109.3)
- moved C5 44.8 mm to (162.2, 109.3)
- moved Q2 44.8 mm to (167.5, 110.6)
- moved Q3 44.8 mm to (184.5, 110.7)
- moved R11 44.8 mm to (162.2, 115.7)
- moved R12 44.8 mm to (173.0, 115.7)
- moved R5 44.8 mm to (179.1, 109.3)
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Other:
- board size 105.4 x 48.9 mm -> 105.4 x 52.1 mm

Commit message: vghnjghj
Parts:
- D2: moved to F.Cu
- moved REF** 11.6 mm to (146.7, 55.9)
- moved JP1 11.4 mm to (129.5, 69.8)
- moved BT1 10.2 mm to (166.4, 73.0)
- moved JP3 7.26 mm to (134.6, 53.3), turned to 90 degrees
- moved J2 3.24 mm to (148.5, 83.8)
- moved J6 3.19 mm to (136.1, 83.8)
- moved JP2 2.62 mm to (127.6, 48.3)
- moved D2 2.54 mm to (129.5, 40.6), turned to 0 degrees

Commit message: dfgdfgd
Parts:
- added REF**: MountingHole_3.2mm_M3_Pad_Via, MountingHole:MountingHole_3.2mm_M3_Pad_Via, F.Cu at (214.6, 86.4)
- C4, C7, D1, J8, J9, Q3, R4, R5, U1: moved to B.Cu
- JP2: value Disable Batt Disconnect -> Batt Sw Disable
- moved REF** 102.6 mm to (214.6, 55.9)
- moved REF** 97.8 mm to (116.8, 86.4)
- moved J9 85.7 mm to (172.1, 84.5), turned to 180 degrees
- moved C4 83.6 mm to (136.9, 71.1), turned to 0 degrees
- moved C7 83.6 mm to (136.9, 74.3), turned to 180 degrees
- moved J5 80.4 mm to (165.1, 86.4)
- moved EC3 77.2 mm to (153.0, 83.4), turned to -90 degrees
- moved J8 76.1 mm to (175.9, 84.5), turned to 180 degrees
- moved U1 68.4 mm to (145.4, 71.1), turned to 180 degrees
- moved EC4 66.4 mm to (154.9, 56.3), turned to -90 degrees
- moved R9 64.9 mm to (143.8, 55.2), turned to 180 degrees
- moved EC5 62.9 mm to (156.8, 70.3), turned to -90 degrees
- moved EC2 61.6 mm to (147.3, 56.1)
- moved R11 61.6 mm to (154.0, 54.6)
- moved R12 59.7 mm to (158.5, 57.8)
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Other:
- board size 105.4 x 52.1 mm -> 105.4 x 50.8 mm

Commit message: yrfthd
Parts:
- moved R12 0.64 mm to (158.4, 57.1)
- turned EC2 to 90 degrees
- turned EC4 to 90 degrees
Routing:
- net GND: track 0.00 -> 305.1 mm, vias 0 -> 5
- net VCC: track 0.00 -> 144.9 mm, vias 0 -> 3
- net Net-(PT4-Pad2): track 0.00 -> 83.7 mm, vias 0 -> 2
- net +BATT: track 0.00 -> 76.2 mm
- net Net-(PT4-Pad1): track 0.00 -> 66.9 mm, vias 0 -> 1
- net Net-(PT3-Pad2): track 0.00 -> 55.7 mm
- net Net-(PT1-Pad2): track 0.00 -> 55.5 mm, vias 0 -> 1
- net /INPUT: track 0.00 -> 50.2 mm
- net -BATT: track 0.00 -> 48.3 mm
- net Net-(EC1-Pad2): track 0.00 -> 45.7 mm
- net /SPKR+: track 0.00 -> 33.8 mm
- net Net-(EC1-Pad1): track 0.00 -> 22.2 mm, vias 0 -> 1
- net /power_in: track 0.00 -> 21.8 mm
- net Net-(EC4-Pad1): track 0.00 -> 20.6 mm
- net Net-(C3-Pad1): track 0.00 -> 20.2 mm
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
Commit message: KJIXCSJIDISDS
Parts:
- C1, C2, C3, C4, C5, C6, C7: footprint Capacitor_SMD:C_0805_2012Metric_Pad1.18x1.45mm_HandSolder -> 000 Capacitors Immo:C_0805_2012Metric_Pad1.18x1.45mm_HandSolder
- JP3: value SWDIR -> SW_DIR
- R1, R10, R11, R12, R13, R2, R3, R4, R5, R6, R7, R8, R9: footprint Resistor_SMD:R_0805_2012Metric_Pad1.20x1.40mm_HandSolder -> 000 Resistors Immo:Resistor_0805_2012_handsolder
- moved R11 1.32 mm to (153.7, 55.9)
- moved R12 1.18 mm to (158.1, 58.3)
- moved Q2 0.76 mm to (161.5, 62.2)
- moved R1 0.63 mm to (153.9, 61.6)
- moved R10 0.63 mm to (158.5, 55.2)
Routing:
- net GND: track 305.1 -> 303.0 mm
- net VCC: track 144.9 -> 146.2 mm
- net Net-(EC4-Pad2): track 4.71 -> 5.72 mm
- net Net-(C5-Pad2): track 12.0 -> 12.8 mm

Commit message: dfgfg
Routing:
- net -BATT: track 48.3 -> 51.0 mm
- added copper zone on B.Cu, net GND
Other:
- board text added: "Gem Toaster Amp"
Changed lines of the file:
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@@
     (fp_line (start 6.985 1.651) (end 6.985 -1.651) (layer "B.SilkS") (width 0.1524))
     (fp_line (start 6.35 -2.286) (end -6.35 -2.286) (layer "B.SilkS") (width 0.1524))
+    (fp_line (start 6.35 2.286) (end -6.35 2.286) (layer "F.SilkS") (width 0.1524))
     (fp_line (start 6.35 -1.651) (end 6.985 -1.651) (layer "F.SilkS") (width 0.1524))
     (fp_line (start 6.35 -2.286) (end 6.35 -1.651) (layer "F.SilkS") (width 0.1524))
@@
     (fp_line (start 6.985 1.651) (end 6.35 1.651) (layer "F.SilkS") (width 0.1524))
     (fp_line (start -6.35 -2.286) (end 6.35 -2.286) (layer "F.SilkS") (width 0.1524))
-    (fp_line (start 6.35 2.286) (end -6.35 2.286) (layer "F.SilkS") (width 0.1524))
     (fp_rect (start -17.78 -2.54) (end 6.985 2.54) (layer "F.SilkS") (width 0.12) (fill none))
     (fp_rect (start -7.112 -2.54) (end 7.112 2.54) (layer "F.CrtYd") (width 0.05) (fill none))
@@
       (effects (font (size 0.5 0.5) (thickness 0.08)))
     )
+    (fp_line (start -0.227064 0.735) (end 0.227064 0.735) (layer "F.SilkS") (width 0.12))
     (fp_line (start -0.227064 -0.735) (end 0.227064 -0.735) (layer "F.SilkS") (width 0.12))
-    (fp_line (start -0.227064 0.735) (end 0.227064 0.735) (layer "F.SilkS") (width 0.12))
     (fp_line (start 1.85 -0.95) (end 1.85 0.95) (layer "F.CrtYd") (width 0.05))
     (fp_line (start -1.85 -0.95) (end 1.85 -0.95) (layer "F.CrtYd") (width 0.05))
+    (fp_line (start -1.85 0.95) (end -1.85 -0.95) (layer "F.CrtYd") (width 0.05))
     (fp_line (start 1.85 0.95) (end -1.85 0.95) (layer "F.CrtYd") (width 0.05))
-    (fp_line (start -1.85 0.95) (end -1.85 -0.95) (layer "F.CrtYd") (width 0.05))
     (fp_line (start 1 -0.625) (end 1 0.625) (layer "F.Fab") (width 0.1))
     (fp_line (start -1 0.625) (end -1 -0.625) (layer "F.Fab") (width 0.1))
@@
       (effects (font (size 0.5 0.5) (thickness 0.08)) (justify mirror))
     )
+    (fp_line (start -0.227064 -0.735) (end 0.227064 -0.735) (layer "B.SilkS") (width 0.12))
     (fp_line (start -0.227064 0.735) (end 0.227064 0.735) (layer "B.SilkS") (width 0.12))
-    (fp_line (start -0.227064 -0.735) (end 0.227064 -0.735) (layer "B.SilkS") (width 0.12))
+    (fp_line (start 1.85 0.95) (end 1.85 -0.95) (layer "B.CrtYd") (width 0.05))
+    (fp_line (start -1.85 0.95) (end 1.85 0.95) (layer "B.CrtYd") (width 0.05))
     (fp_line (start 1.85 -0.95) (end -1.85 -0.95) (layer "B.CrtYd") (width 0.05))
-    (fp_line (start 1.85 0.95) (end 1.85 -0.95) (layer "B.CrtYd") (width 0.05))
     (fp_line (start -1.85 -0.95) (end -1.85 0.95) (layer "B.CrtYd") (width 0.05))
-    (fp_line (start -1.85 0.95) (end 1.85 0.95) (layer "B.CrtYd") (width 0.05))
     (fp_line (start 1 -0.625) (end -1 -0.625) (layer "B.Fab") (width 0.1))
     (fp_line (start 1 0.625) (end 1 -0.625) (layer "B.Fab") (width 0.1))
@@
   (gr_line (start 218.44 43.18) (end 218.44 86.36) (layer "Edge.Cuts") (width 0.1))
   (gr_line (start 214.63 90.17) (end 116.84 90.17) (layer "Edge.Cuts") (width 0.1))
+  (gr_text "Gem Toaster Amp" (at 184.785 68.58) (layer "F.SilkS")
+    (effects (font (size 2 2) (thickness 0.3)))
+  )
   (dimension (type aligned) (layer "F.Fab")
     (pts (xy 223.2 30.3006) (xy 223.2 129.3606))
@@
   (segment (start 129.29 48.925) (end 131.165 50.8) (width 1) (layer "F.Cu") (net 1))
   (segment (start 127.635 48.925) (end 129.29 48.925) (width 1) (layer "F.Cu") (net 1))
-  (segment (start 166.37 52.705) (end 164.465 50.8) (width 1) (layer "B.Cu") (net 1))
-  (segment (start 164.465 50.8) (end 131.165 50.8) (width 1) (layer "B.Cu") (net 1))
   (segment (start 166.37 60.325) (end 166.37 52.705) (width 1) (layer "B.Cu") (net 1))
+  (segment (start 166.37 52.705) (end 161.29 47.625) (width 1) (layer "B.Cu") (net 1))
+  (segment (start 161.29 47.625) (end 134.34 47.625) (width 1) (layer "B.Cu") (net 1))
+  (segment (start 134.34 47.625) (end 131.165 50.8) (width 1) (layer "B.Cu") (net 1))
   (segment (start 128.24 71.755) (end 122.694511 77.300489) (width 1) (layer "F.Cu") (net 2))
   (segment (start 128.24 71.755) (end 128.24 66.705) (width 1) (layer "F.Cu") (net 2))
@@
   (segment (start 134.62 54.61) (end 134.62 57.15) (width 1) (layer "F.Cu") (net 32))
   (segment (start 134.62 57.15) (end 138.43 60.96) (width 1) (layer "F.Cu") (net 32))
+  (zone (net 8) (net_name "GND") (layer "B.Cu") (hatch edge 0.508)
+    (connect_pads (clearance 0.508))
+    (min_thickness 0.254) (filled_areas_thickness no)
+    (fill yes (thermal_gap 0.508) (thermal_bridge_width 0.508))
+    (polygon
+      (pts
+        (xy 219.075 90.805)
+        (xy 112.395 90.805)
+        (xy 112.395 38.735)
+        (xy 219.075 38.735)
+      )
+    )
+  )
 )

Commit message: sadf
Parts:
- JP2: value Batt Sw Disable -> Batt Sw Bypass
- moved J3 2.54 mm to (115.6, 69.8), turned to -90 degrees
Routing:
- net /INPUT: track 50.2 -> 52.0 mm
- net GND: track 303.0 -> 304.1 mm
Other:
- board text added: "Design By:"
- board text added: "ImogenWren"
- board text added: "Unit No:"
- board text added: "github.com/ImogenWren github.com/PanGalacticTech PanGalacticTech.com/"
