File: GemToasterAmp.kicad_pcb (KiCad board)
At the start: 2 copper layers, 105.4 x 50.8 mm, 53 parts, among them J1 Input, J2 Speaker(2-8 ohm), J3 Input, J5 Speaker, J6 Power, J7 AudioJack3_Switch, J8 Vcc, J9 GND, Q1 2N5457/J201, Q2 2N5457/J201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

Commit message: added gerbers
Parts:
- added REF**: OSHW-Logo2_9.8x8mm_Copper, Symbol:OSHW-Logo2_9.8x8mm_Copper, F.Cu at (212.7, 64.1)
- added REF**: KiCad-Logo_6mm_Copper, Symbol:KiCad-Logo_6mm_Copper, F.Cu at (126.4, 46.4)
- PT1, PT2, PT3, PT4: footprint 000 Resistors Immo:16MM_AngleMount -> 000_Resistors_Immo:16MM_AngleMount
- U1: footprint 000 IC Immo:DIL8 -> 000_ICs_Immo:DIL8
Other:
- board text added: "Design By: ImogenWren"

Commit message: gvhjng
Parts:
- removed the REF** at (126.4, 46.4)
Other:
- board text added: "JLCJLCJLCJLC"
